Commit message: [update] portable station for gazebo

File: mimik_ur3_lab_mobile_moveit_config/config/gazebo_mimik_ur3_station_portable.urdf (robot description, URDF)
Before this commit: robot mimik_ur3_station_portable, 39 links, 38 joints
Links:
- added link robotiq_2f140_left_fingertip_pad, mass 0.0212636185801172; collision mesh filename=package://robotiq_description/meshes/robotiq_agc_tip_220_14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; visual mesh filename=package://robotiq_description/meshes/robotiq_agc_tip_220_14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
- added link robotiq_2f140_right_fingertip_pad, mass 0.0212636185801172; collision mesh filename=package://robotiq_description/meshes/robotiq_agc_tip_220_14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; visual mesh filename=package://robotiq_description/meshes/robotiq_agc_tip_220_14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
- link newport_base: geometry collision mesh filename=package://mimik_description/meshes/newport/sa2_30x30/collis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; visual mesh filename=package://mimik_description/meshes/newport/sa2_30x30/visual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
- link pipette_base: geometry collision mesh filename=package://mimik_description/meshes/mimik/pipette_p200/colli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; visual mesh filename=package://mimik_description/meshes/mimik/pipette_p200/visua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
- link tabletop: geometry collision box size=1.1176 1.27 0.0254
- link ur3_base_link_inertia: geometry collision mesh filename=package://ur_description/meshes/ur3/collision/vhacd_h16/bas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; visual mesh filename=package://ur_description/meshes/ur3/visual/base.dae
- link ur3_forearm_link: geometry collision mesh filename=package://ur_description/meshes/ur3/collision/vhacd_h16/for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; visual mesh filename=package://ur_description/meshes/ur3/visual/forearm.dae
- link ur3_mounting_plate_base: geometry collision mesh filename=package://mimik_description/meshes/mimik/ur3_mounting_plate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; visual mesh filename=package://mimik_description/meshes/mimik/ur3_mounting_plate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
- link ur3_shoulder_link: geometry collision mesh filename=package://ur_description/meshes/ur3/collision/vhacd_h16/sho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; visual mesh filename=package://ur_description/meshes/ur3/visual/shoulder.dae
- link ur3_upper_arm_link: geometry collision mesh filename=package://ur_description/meshes/ur3/collision/vhacd_h16/upp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; visual mesh filename=package://ur_description/meshes/ur3/visual/upperarm.dae
- link ur3_wrist_1_link: geometry collision mesh filename=package://ur_description/meshes/ur3/collision/vhacd_h16/wri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; visual mesh filename=package://ur_description/meshes/ur3/visual/wrist1.dae
- link ur3_wrist_2_link: geometry collision mesh filename=package://ur_description/meshes/ur3/collision/vhacd_h16/wri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; visual mesh filename=package://ur_description/meshes/ur3/visual/wrist2.dae
- link ur3_wrist_3_link: geometry collision mesh filename=package://ur_description/meshes/ur3/collision/vhacd_h16/wri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; visual mesh filename=package://ur_description/meshes/ur3/visual/wrist3.dae
- link wall: geometry collision box size=1.1176 1.27 0.0254
Joints:
- added joint robotiq_2f140_left_fingertip_pad_joint: type fixed, parent robotiq_2f140_left_fingertip, child robotiq_2f140_left_fingertip_pad, origin xyz=0 0.00476 0  rpy=0 0 0
- added joint robotiq_2f140_right_fingertip_pad_joint: type fixed, parent robotiq_2f140_right_fingertip, child robotiq_2f140_right_fingertip_pad, origin xyz=0 0.00476 0  rpy=0 0 0
- joint robotiq_2f140_base_joint: origin xyz=0.0 0.0 0.0 rpy=0.0 0.0 0.0 -> xyz=0.0010977079105917165 -0.00047849967130053628 -2.3860966923898729e-05 rpy=0 0 0
- joint robotiq_2f140_left_inner_finger_joint: mimic (none) -> joint=robotiq_2f140_left_outer_knuckle_joint multiplier=-1 offset=0
- joint robotiq_2f140_left_inner_knuckle_joint: mimic (none) -> joint=robotiq_2f140_left_outer_knuckle_joint multiplier=1 offset=0
- joint robotiq_2f140_right_inner_finger_joint: mimic (none) -> joint=robotiq_2f140_left_outer_knuckle_joint multiplier=-1 offset=0
- joint robotiq_2f140_right_inner_knuckle_joint: mimic (none) -> joint=robotiq_2f140_left_outer_knuckle_joint multiplier=1 offset=0
- joint robotiq_2f140_right_outer_knuckle_joint: mimic (none) -> joint=robotiq_2f140_left_outer_knuckle_joint multiplier=1 offset=0
- joint robotiq_ft300_frame_id_joint: origin xyz=0 0 0 rpy=-1.5707963267948966 0 -1.5707963267948966 -> xyz=0.0348 0 0 rpy=-1.5707963267948966 0 -1.5707963267948966
- joint robotiq_ft300_toolside_joint: origin xyz=0.0348 0 0 rpy=0 0 0 -> xyz=0 0 0 rpy=0 -1.5707963267948966 1.5707963267948966; parent robotiq_ft300_robotside -> robotiq_ft300_frame_id
- joint ur3_mounting_plate_base_joint: origin xyz=-0.254 -0.30479999999999996 0.0 rpy=0.0 0.0 0.0 -> xyz=-0.0508 0.07619999999999999 0.0 rpy=0.0 0.0 -1.5707963267948966
- joint wall_joint: origin xyz=0 -0.5460999999999999 0.5588 rpy=0.0 0.0 0.0 -> xyz=-0.5460999999999999 0 0.5588 rpy=0.0 0.0 0.0
