Commit message: [fix] removed labware

File: mimik_ur3_setup_description/urdf/mimik_ur3_lab_mobile.xacro (robot description, xacro)
@@ -53,8 +53,4 @@
   <xacro:newport_sa2_30x30
     prefix="newport_"/>
-  <xacro:mimik_biorad_t100_adapter
-    prefix="t100_adapter_"/>
-  <xacro:biorad_thermal_cycler_t100_open
-    prefix="t100_"/>
   <xacro:mimik_ur3_mounting_plate
     prefix="ur3_mounting_plate_"/>
@@ -100,16 +96,4 @@
     <origin xyz="${-2 * 0.0254} ${12 * 0.0254} 0.0" rpy="0.0 0.0 ${-pi/2}" />
   </joint>
-  <joint name="t100_adapter_joint" type="fixed">
-    <parent link= "newport_tabletop" />
-    <child link = "t100_adapter_base" />
-    <!-- Newport tabletop has matrix of 1 inch hole gap-->
-    <origin xyz="${-3.5 * 0.0254} ${-4.5 * 0.0254} 0.0" rpy="0.0 0.0 ${0.927295218}" />
-  </joint>
-  <joint name="t100_joint" type="fixed">
-    <parent link= "t100_adapter_base" />
-    <child link = "t100_base" />
-    <!-- Newport tabletop has matrix of 1 inch hole gap-->
-    <origin xyz="0.0 0.0 0.0" rpy="0.0 0.0 0.0" />
-  </joint>
   <joint name="ur3_base_joint" type="fixed">
     <parent link= "ur3_mounting_plate_robotside" />

Commit message: [config] add the realsense camera and adapter to the URDF

File: mimik_ur3_setup_description/urdf/mimik_ur3_lab_mobile.xacro (robot description, xacro)
@@ -12,4 +12,7 @@
   <xacro:include filename="$(find mimik_description)/urdf/mimik/biorad_t100_adapter_macro.xacro"/>
   <xacro:include filename="$(find mimik_description)/urdf/biorad/thermal_cycler_t100_open_macro.xacro"/>
+  <xacro:include filename="$(find mimik_description)/urdf/picknik/ur5_realsense_camera_adapter_macro.xacro"/>
+  <!-- <xacro:include filename="$(find mimik_description)/urdf/intel/realsense_d415_macro.xacro"/> -->
+  <xacro:include filename="$(find realsense2_description)/urdf/_d415.urdf.xacro" />
   <!-- TCP calibration of the robotiq gripper (xyz)-->
   <xacro:property name="tcp_calibration_gripper" value="0.0010977079105917165 -0.00047849967130053628 -2.3860966923898729e-05" />
@@ -71,4 +74,11 @@
     prefix="dual_gripper_coupling_"
     visual_parameters_file="$(find robotiq_description)/config/robotiq_agc_apl_159_002/visual_parameters_bbox.yaml"/>
+  <!-- Realsense D415 adapter -->
+  <xacro:picknik_ur5_realsense_camera_adapter
+    prefix="camera_adapter_"/>
+  <!-- Realsense D415 camera -->
+  <xacro:sensor_d415 parent="camera_adapter_camera" name="camera" use_nominal_extrinsics="false" add_plug="true" use_mesh="true">
+    <origin xyz="${0.02005/2} 0 ${-0.023/2}" rpy="0 0 0"/>
+  </xacro:sensor_d415>
   <!-- 2f-140 gripper + sillicon fingertip pads -->
   <xacro:robotiq_2f_140
@@ -117,6 +127,16 @@
     <origin xyz="0.0 0.0 0.0" rpy="0.0 0.0 0.0" />
   </joint>
+  <joint name="camera_adapter_robotside_joint" type="fixed">
+    <parent link= "dual_gripper_coupling_toolside_left" />
+    <child link = "camera_adapter_robotside" />
+    <origin xyz="0 0 0" rpy="0 0 0" />
+  </joint>
+  <!-- <joint name="camera_backside_joint" type="fixed"> -->
+  <!--   <parent link= "camera_adapter_camera" /> -->
+  <!--   <child link = "camera_backside" /> -->
+  <!--   <origin xyz="0 0 0" rpy="0 0 0" /> -->
+  <!-- </joint> -->
   <joint name="robotiq_2f140_base_joint" type="fixed">
-    <parent link= "dual_gripper_coupling_toolside_left" />
+    <parent link= "camera_adapter_toolside" />
     <child link = "robotiq_2f140_base_link" />
     <!-- <origin xyz="0.0 0.0 0.0" rpy="0 0 0" /> -->

Commit message: [config] move ur3 base to center of table

File: mimik_ur3_setup_description/urdf/mimik_ur3_lab_mobile.xacro (robot description, xacro)
@@ -104,5 +104,5 @@
     <child link = "ur3_mounting_plate_base" />
     <!-- Newport tabletop has matrix of 1 inch hole gap-->
-    <origin xyz="${-2 * 0.0254} ${12 * 0.0254} 0.0" rpy="0.0 0.0 ${-pi/2}" />
+    <origin xyz="${-2 * 0.0254} ${3 * 0.0254} 0.0" rpy="0.0 0.0 ${-pi/2}" />
   </joint>
   <joint name="ur3_base_joint" type="fixed">

Commit message: [update] pipette xacro changes

File: mimik_ur3_setup_description/urdf/mimik_ur3_lab_mobile.xacro (robot description, xacro)
@@ -145,5 +145,5 @@
   <joint name="pipette_base_joint" type="fixed">
     <parent link= "dual_gripper_coupling_toolside_right" />
-    <child link = "pipette_base" />
+    <child link = "pipette_robotside" />
     <origin xyz="0.0 0.0 0.0" rpy="0.0 0.0 0.0" />
   </joint>

Commit message: [update] change newport frame orientation

File: mimik_ur3_setup_description/urdf/mimik_ur3_lab_mobile.xacro (robot description, xacro)
@@ -98,5 +98,5 @@
     <parent link= "tabletop" />
     <child link = "wall" />
-    <origin xyz="${-(22 * 0.0254 - 0.0254/2)} 0 ${44*0.0254/2}" rpy="0.0 0.0 0.0" />
+    <origin xyz="${(22 * 0.0254 - 0.0254/2)} 0 ${44*0.0254/2}" rpy="0.0 0.0 0.0" />
   </joint>
   <joint name="ur3_mounting_plate_base_joint" type="fixed">
@@ -104,5 +104,5 @@
     <child link = "ur3_mounting_plate_base" />
     <!-- Newport tabletop has matrix of 1 inch hole gap-->
-    <origin xyz="${-2 * 0.0254} ${3 * 0.0254} 0.0" rpy="0.0 0.0 ${-pi/2}" />
+    <origin xyz="${2 * 0.0254} ${-3 * 0.0254}  0.0" rpy="0.0 0.0 ${pi/2}" />
   </joint>
   <joint name="ur3_base_joint" type="fixed">

Commit message: [impl] tcp pipette calibration

File: mimik_ur3_setup_description/urdf/mimik_ur3_lab_mobile.xacro (robot description, xacro)
@@ -81,4 +81,5 @@
     <origin xyz="${0.02005/2} 0 ${-0.023/2}" rpy="0 0 0"/>
   </xacro:sensor_d415>
+  <link name="pipette_tcp" />
   <!-- 2f-140 gripper + sillicon fingertip pads -->
   <xacro:robotiq_2f_140
@@ -146,4 +147,12 @@
     <parent link= "dual_gripper_coupling_toolside_right" />
     <child link = "pipette_robotside" />
+    <!-- Calibrated on Jan 21 2024 -->
+    <!-- Offset the hole pipette CAD wrt. the calibrated tcp of the tip -->
+    <origin xyz="${0.25519783013035285 - 0.253442} -0.00026130058471244416 -0.0008577228691093923" rpy="0.0 0.0 0.0" />
+  </joint>
+  <!-- Conveniance frame -->
+  <joint name="pipette_tcp_joint" type="fixed">
+    <parent link= "pipette_tip" />
+    <child link = "pipette_tcp" />
     <origin xyz="0.0 0.0 0.0" rpy="0.0 0.0 0.0" />
   </joint>

Commit message: [fix] tcp calibration is not needed with the new base

File: mimik_ur3_setup_description/urdf/mimik_ur3_lab_mobile.xacro (robot description, xacro)
@@ -16,5 +16,6 @@
   <xacro:include filename="$(find realsense2_description)/urdf/_d415.urdf.xacro" />
   <!-- TCP calibration of the robotiq gripper (xyz)-->
-  <xacro:property name="tcp_calibration_gripper" value="0.0010977079105917165 -0.00047849967130053628 -2.3860966923898729e-05" />
+  <!-- <xacro:property name="tcp_calibration_gripper" value="0.0010977079105917165 -0.00047849967130053628 -2.3860966923898729e-05" /> -->
+  <xacro:property name="tcp_calibration_gripper" value="0.0 0.0 0.0" />
   <!-- Table supporting the tabletop breadboard -->
   <link name="tabletop">

Commit message: [fix] wrong child link

File: mimik_ur3_setup_description/urdf/mimik_ur3_lab_mobile.xacro (robot description, xacro)
@@ -147,5 +147,5 @@
   <joint name="pipette_base_joint" type="fixed">
     <parent link= "dual_gripper_coupling_toolside_right" />
-    <child link = "pipette_robotside" />
+    <child link = "pipette_base" />
     <!-- Calibrated on Jan 21 2024 -->
     <!-- Offset the hole pipette CAD wrt. the calibrated tcp of the tip -->

Commit message: [refac] drop the real-sense for the moment

File: mimik_ur3_setup_description/urdf/mimik_ur3_lab_mobile.xacro (robot description, xacro)
@@ -75,12 +75,12 @@
     prefix="dual_gripper_coupling_"
     visual_parameters_file="$(find robotiq_description)/config/robotiq_agc_apl_159_002/visual_parameters_bbox.yaml"/>
-  <!-- Realsense D415 adapter -->
-  <xacro:picknik_ur5_realsense_camera_adapter
-    prefix="camera_adapter_"/>
-  <!-- Realsense D415 camera -->
-  <xacro:sensor_d415 parent="camera_adapter_camera" name="camera" use_nominal_extrinsics="false" add_plug="true" use_mesh="true">
-    <origin xyz="${0.02005/2} 0 ${-0.023/2}" rpy="0 0 0"/>
-  </xacro:sensor_d415>
   <link name="pipette_tcp" />
+  <!-- <!-\- Realsense D415 adapter -\-> -->
+  <!-- <xacro:picknik_ur5_realsense_camera_adapter -->
+  <!--   prefix="camera_adapter_"/> -->
+  <!-- <!-\- Realsense D415 camera -\-> -->
+  <!-- <xacro:sensor_d415 parent="camera_adapter_camera" name="camera" use_nominal_extrinsics="false" add_plug="true" use_mesh="true"> -->
+  <!--   <origin xyz="${0.02005/2} 0 ${-0.023/2}" rpy="0 0 0"/> -->
+  <!-- </xacro:sensor_d415> -->
   <!-- 2f-140 gripper + sillicon fingertip pads -->
   <xacro:robotiq_2f_140
@@ -129,16 +129,17 @@
     <origin xyz="0.0 0.0 0.0" rpy="0.0 0.0 0.0" />
   </joint>
-  <joint name="camera_adapter_robotside_joint" type="fixed">
-    <parent link= "dual_gripper_coupling_toolside_left" />
-    <child link = "camera_adapter_robotside" />
-    <origin xyz="0 0 0" rpy="0 0 0" />
-  </joint>
-  <!-- <joint name="camera_backside_joint" type="fixed"> -->
-  <!--   <parent link= "camera_adapter_camera" /> -->
-  <!--   <child link = "camera_backside" /> -->
+  <!-- <joint name="camera_adapter_robotside_joint" type="fixed"> -->
+  <!--   <parent link= "dual_gripper_coupling_toolside_left" /> -->
+  <!--   <child link = "camera_adapter_robotside" /> -->
   <!--   <origin xyz="0 0 0" rpy="0 0 0" /> -->
   <!-- </joint> -->
+  <!-- <joint name="robotiq_2f140_base_joint" type="fixed"> -->
+  <!--   <parent link= "camera_adapter_toolside" /> -->
+  <!--   <child link = "robotiq_2f140_base_link" /> -->
+  <!--   <!-\- <origin xyz="0.0 0.0 0.0" rpy="0 0 0" /> -\-> -->
+  <!--   <origin xyz="${tcp_calibration_gripper}" rpy="0 0 0" /> -->
+  <!-- </joint> -->
   <joint name="robotiq_2f140_base_joint" type="fixed">
-    <parent link= "camera_adapter_toolside" />
+    <parent link= "dual_gripper_coupling_toolside_left" />
     <child link = "robotiq_2f140_base_link" />
     <!-- <origin xyz="0.0 0.0 0.0" rpy="0 0 0" /> -->

Commit message: [impl] add gripper tcp calibration

File: mimik_ur3_setup_description/urdf/mimik_ur3_lab_mobile.xacro (robot description, xacro)
@@ -17,5 +17,6 @@
   <!-- TCP calibration of the robotiq gripper (xyz)-->
   <!-- <xacro:property name="tcp_calibration_gripper" value="0.0010977079105917165 -0.00047849967130053628 -2.3860966923898729e-05" /> -->
-  <xacro:property name="tcp_calibration_gripper" value="0.0 0.0 0.0" />
+  <!-- wrt. the robotiq_base frame -->
+  <xacro:property name="tcp_calibration_gripper" value="0.00160516037 0.00101565847 -0.00215532428" />
   <!-- Table supporting the tabletop breadboard -->
   <link name="tabletop">

Commit message: [refac] use ur3 big mounting plate

File: mimik_ur3_setup_description/urdf/mimik_ur3_lab_mobile.xacro (robot description, xacro)
@@ -2,5 +2,5 @@
 <robot name="mimik_ur3_station_portable" xmlns:xacro="http://ros.org/wiki/xacro" >
   <xacro:include filename="$(find mimik_description)/urdf/newport/sa2_30x30_macro.xacro"/>
-  <xacro:include filename="$(find mimik_description)/urdf/mimik/ur3_mounting_plate_macro.xacro"/>
+  <xacro:include filename="$(find mimik_description)/urdf/mimik/ur3_big_mounting_plate_macro.xacro"/>
   <xacro:include filename="$(find ur_description)/urdf/inc/ur3_macro.xacro"/>
   <xacro:include filename="$(find robotiq_description)/urdf/robotiq_fts_300_cpl_062/robotiq_fts_300_cpl_062_macro.xacro"/>
@@ -58,5 +58,5 @@
   <xacro:newport_sa2_30x30
     prefix="newport_"/>
-  <xacro:mimik_ur3_mounting_plate
+  <xacro:mimik_ur3_big_mounting_plate
     prefix="ur3_mounting_plate_"/>
   <!-- UR3 with S/N: 2017333047 -->
@@ -107,10 +107,10 @@
     <child link = "ur3_mounting_plate_base" />
     <!-- Newport tabletop has matrix of 1 inch hole gap-->
-    <origin xyz="${2 * 0.0254} ${-3 * 0.0254}  0.0" rpy="0.0 0.0 ${pi/2}" />
+    <origin xyz="${2 * 0.0254} ${-3 * 0.0254}  0.0" rpy="0.0 0.0 0.0" />
   </joint>
   <joint name="ur3_base_joint" type="fixed">
     <parent link= "ur3_mounting_plate_robotside" />
     <child link = "ur3_base_link" />
-    <origin xyz="0.0 0.0 0.0" rpy="0.0 0.0 0.0" />
+    <origin xyz="0.0 0.0 0.0" rpy="0.0 0.0 ${pi/2}" />
   </joint>
   <joint name="robotiq_fts300_coupling_joint" type="fixed">

Commit message: [impl] added realsense camera to setup

File: mimik_ur3_setup_description/urdf/mimik_ur3_lab_mobile.xacro (robot description, xacro)
@@ -77,11 +77,11 @@
     visual_parameters_file="$(find robotiq_description)/config/robotiq_agc_apl_159_002/visual_parameters_bbox.yaml"/>
   <link name="pipette_tcp" />
-  <!-- <!-\- Realsense D415 adapter -\-> -->
-  <!-- <xacro:picknik_ur5_realsense_camera_adapter -->
-  <!--   prefix="camera_adapter_"/> -->
-  <!-- <!-\- Realsense D415 camera -\-> -->
-  <!-- <xacro:sensor_d415 parent="camera_adapter_camera" name="camera" use_nominal_extrinsics="false" add_plug="true" use_mesh="true"> -->
-  <!--   <origin xyz="${0.02005/2} 0 ${-0.023/2}" rpy="0 0 0"/> -->
-  <!-- </xacro:sensor_d415> -->
+  <!-- Realsense D415 adapter -->
+  <xacro:picknik_ur5_realsense_camera_adapter
+    prefix="camera_adapter_"/>
+  <!-- Realsense D415 camera -->
+  <xacro:sensor_d415 parent="camera_adapter_camera" name="camera" use_nominal_extrinsics="false" add_plug="true" use_mesh="true">
+    <origin xyz="${0.02005/2} 0 ${-0.023/2}" rpy="0 0 0"/>
+  </xacro:sensor_d415>
   <!-- 2f-140 gripper + sillicon fingertip pads -->
   <xacro:robotiq_2f_140
@@ -130,20 +130,26 @@
     <origin xyz="0.0 0.0 0.0" rpy="0.0 0.0 0.0" />
   </joint>
-  <!-- <joint name="camera_adapter_robotside_joint" type="fixed"> -->
+  <joint name="camera_adapter_robotside_joint" type="fixed">
+    <parent link= "dual_gripper_coupling_toolside_left" />
+    <child link = "camera_adapter_robotside" />
+    <origin xyz="0 0 0" rpy="0 0 0" />
+  </joint>
+  <joint name="robotiq_2f140_base_joint" type="fixed">
+    <parent link= "camera_adapter_toolside" />
+    <child link = "robotiq_2f140_base_link" />
+    <!-- <origin xyz="0.0 0.0 0.0" rpy="0 0 0" /> -->
+    <origin xyz="${tcp_calibration_gripper}" rpy="0 0 0" />
+  </joint>
+  <!-- <joint name="robotiq_2f140_base_joint" type="fixed"> -->
   <!--   <parent link= "dual_gripper_coupling_toolside_left" /> -->
-  <!--   <child link = "camera_adapter_robotside" /> -->
-  <!--   <origin xyz="0 0 0" rpy="0 0 0" /> -->
-  <!-- </joint> -->
-  <!-- <joint name="robotiq_2f140_base_joint" type="fixed"> -->
-  <!--   <parent link= "camera_adapter_toolside" /> -->
   <!--   <child link = "robotiq_2f140_base_link" /> -->
   <!--   <!-\- <origin xyz="0.0 0.0 0.0" rpy="0 0 0" /> -\-> -->
   <!--   <origin xyz="${tcp_calibration_gripper}" rpy="0 0 0" /> -->
   <!-- </joint> -->
-  <joint name="robotiq_2f140_base_joint" type="fixed">
+  <link name="robotiq_2f140_tcp_cad"/>
+  <joint name="robotiq_2f140_tcp_cad_joint" type="fixed">
     <parent link= "dual_gripper_coupling_toolside_left" />
-    <child link = "robotiq_2f140_base_link" />
-    <!-- <origin xyz="0.0 0.0 0.0" rpy="0 0 0" /> -->
-    <origin xyz="${tcp_calibration_gripper}" rpy="0 0 0" />
+    <child link = "robotiq_2f140_tcp_cad" />
+    <origin xyz="0.24127678495 0 0" rpy="0 0 0" />
   </joint>
   <joint name="pipette_base_joint" type="fixed">

Commit message: [impl] camera color calibration link

File: mimik_ur3_setup_description/urdf/mimik_ur3_lab_mobile.xacro (robot description, xacro)
@@ -84,4 +84,5 @@
     <origin xyz="${0.02005/2} 0 ${-0.023/2}" rpy="0 0 0"/>
   </xacro:sensor_d415>
+  <link name="camera_color_optical_frame"/>
   <!-- 2f-140 gripper + sillicon fingertip pads -->
   <xacro:robotiq_2f_140
@@ -141,4 +142,10 @@
     <origin xyz="${tcp_calibration_gripper}" rpy="0 0 0" />
   </joint>
+  <!-- Calibrated -->
+  <joint name="camera_color_optical_frame_joint" type="fixed">
+    <parent link= "ur3_wrist_3_link" />
+    <child link = "camera_color_optical_frame" />
+   <origin xyz="-0.0885371 -0.0804488 0.058979" rpy="2.95938 -2.36642 3.00636" />
+  </joint>
   <!-- <joint name="robotiq_2f140_base_joint" type="fixed"> -->
   <!--   <parent link= "dual_gripper_coupling_toolside_left" /> -->

Commit message: [fix] rpy calibration error
https://github.com/ros-planning/moveit_calibration/issues/132

File: mimik_ur3_setup_description/urdf/mimik_ur3_lab_mobile.xacro (robot description, xacro)
@@ -142,9 +142,10 @@
     <origin xyz="${tcp_calibration_gripper}" rpy="0 0 0" />
   </joint>
-  <!-- Calibrated -->
+  <!-- Calibrated with moveit_calibration pkg -->
+  <!-- Error: 0.0021 m, 0.0063 rad-->
   <joint name="camera_color_optical_frame_joint" type="fixed">
     <parent link= "ur3_wrist_3_link" />
     <child link = "camera_color_optical_frame" />
-   <origin xyz="-0.0885371 -0.0804488 0.058979" rpy="2.95938 -2.36642 3.00636" />
+    <origin xyz="-0.0852237 -0.0776651 0.0608126" rpy="-0.1188682 -0.7931895 -0.0029631" />
   </joint>
   <!-- <joint name="robotiq_2f140_base_joint" type="fixed"> -->

Commit message: [refac] update pipette tcp calibration

File: mimik_ur3_setup_description/urdf/mimik_ur3_lab_mobile.xacro (robot description, xacro)
@@ -164,13 +164,23 @@
     <parent link= "dual_gripper_coupling_toolside_right" />
     <child link = "pipette_base" />
-    <!-- Calibrated on Jan 21 2024 -->
-    <!-- Offset the hole pipette CAD wrt. the calibrated tcp of the tip -->
-    <origin xyz="${0.25519783013035285 - 0.253442} -0.00026130058471244416 -0.0008577228691093923" rpy="0.0 0.0 0.0" />
+    <origin xyz="0.0 0.0 0.0" rpy="${pi} 0.0 0.0" />
   </joint>
+  <!-- Sanity Check -->
+  <!-- <link name="pipette_tcp_test"/> -->
+  <!-- <joint name="lol" type="fixed"> -->
+  <!--   <parent link= "ur3_tool0" /> -->
+  <!--   <child link = "pipette_tcp_test" /> -->
+  <!--   <origin xyz="0.223439 -0.00046209 0.243363" rpy="0.0 0.0 0.0" /> -->
+  <!-- </joint> -->
   <!-- Conveniance frame -->
   <joint name="pipette_tcp_joint" type="fixed">
     <parent link= "pipette_tip" />
     <child link = "pipette_tcp" />
-    <origin xyz="0.0 0.0 0.0" rpy="0.0 0.0 0.0" />
+    <!-- Calibrated on Apr 18 2024 with Tool Point Calibration ROS package -->
+    <!-- Calibration captured 4 tool poses (out of 4 requested). Computing calibration... -->
+    <!-- Calibrated tcp (meters in xyz): [   0.223439 -0.00046209    0.243363] from ur3_tool0 -->
+    <!-- Touch point (meters in xyz): [-0.240945  0.241088 0.0427421] in frame newport_tabletop -->
+    <!-- Average residual: 1.43073e-07 -->
+    <origin xyz="0.0006228806938889386 0.0011144002871499858 -0.00046208999999987344" rpy="0.0 0.0 0.0" />
   </joint>
 </robot>

Commit message: [refac] update calibration

File: mimik_ur3_setup_description/urdf/mimik_ur3_lab_mobile.xacro (robot description, xacro)
@@ -182,5 +182,6 @@
     <!-- Touch point (meters in xyz): [-0.240945  0.241088 0.0427421] in frame newport_tabletop -->
     <!-- Average residual: 1.43073e-07 -->
-    <origin xyz="0.0006228806938889386 0.0011144002871499858 -0.00046208999999987344" rpy="0.0 0.0 0.0" />
+    <!-- <origin xyz="0.0006228806938889386 0.0011144002871499858 -0.00046208999999987344" rpy="0.0 0.0 0.0" /> -->
+    <origin xyz="0.0006464523002427391 0.0005510077330404747 -0.0007046087554606569" rpy="${pi} 0.0 0.0" />
   </joint>
 </robot>
