Commit message: Use new realsense camera adapter
Reconfigured with moveit setup assistant.

File: mimik_ur3_setup_description/urdf/mimik_ur3_lab3023.xacro (robot description, xacro)
@@ -10,4 +10,5 @@
   <xacro:include filename="$(find robotiq_description)/urdf/robotiq_agc_tip_220_140/robotiq_agc_tip_220_140_macro.xacro"/>
   <xacro:include filename="$(find mimik_description)/urdf/mimik/pipette_p200_macro.xacro"/>
+  <xacro:include filename="$(find mimik_description)/urdf/mimik/realsense_camera_adapter_macro.xacro"/>
   <xacro:include filename="$(find mimik_description)/urdf/mimik/biorad_t100_adapter_macro.xacro"/>
   <xacro:include filename="$(find mimik_description)/urdf/biorad/thermocycler_t100_open_macro.xacro"/>
@@ -77,9 +78,9 @@
     visual_parameters_file="$(find robotiq_description)/config/robotiq_agc_apl_159_002/visual_parameters_bbox.yaml"/>
   <link name="pipette_tcp" />
-  <!-- Realsense D415 adapter -->
-  <xacro:picknik_ur5_realsense_camera_adapter
+  <!-- Mimik camera adapter attached to gripper -->
+  <xacro:mimik_realsense_camera_adapter
     prefix="camera_adapter_"/>
   <!-- Realsense D415 camera -->
-  <xacro:sensor_d415 parent="camera_adapter_camera" name="camera" use_nominal_extrinsics="false" add_plug="true" use_mesh="true">
+  <xacro:sensor_d415 parent="camera_adapter_toolside" name="camera" use_nominal_extrinsics="false" add_plug="true" use_mesh="true">
     <origin xyz="${0.02005/2} 0 ${-0.023/2}" rpy="0 0 0"/>
   </xacro:sensor_d415>
@@ -141,14 +142,14 @@
     <origin xyz="0.0 0.0 0.0" rpy="0.0 0.0 0.0" />
   </joint>
-  <joint name="camera_adapter_robotside_joint" type="fixed">
+  <joint name="robotiq_2f140_base_joint" type="fixed">
     <parent link= "dual_gripper_coupling_toolside_left" />
-    <child link = "camera_adapter_robotside" />
-    <origin xyz="0 0 0" rpy="0 0 0" />
-  </joint>
-  <joint name="robotiq_2f140_base_joint" type="fixed">
-    <parent link= "camera_adapter_toolside" />
     <child link = "robotiq_2f140_base_link" />
     <!-- <origin xyz="0.0 0.0 0.0" rpy="0 0 0" /> -->
     <origin xyz="${tcp_calibration_gripper}" rpy="0 0 0" />
+  </joint>
+  <joint name="camera_adapter_robotside_joint" type="fixed">
+    <parent link= "robotiq_2f140_base_link" />
+    <child link = "camera_adapter_robotside" />
+    <origin xyz="0.0443 0 0.0385" rpy="0 0 0" />
   </joint>
   <!-- Calibrated with moveit_calibration pkg -->

Commit message: Use theoritical rgb camera pose

File: mimik_ur3_setup_description/urdf/mimik_ur3_lab3023.xacro (robot description, xacro)
@@ -155,8 +155,14 @@
   <!-- Calibrated with moveit_calibration pkg -->
   <!-- Error: 0.0021 m, 0.0063 rad-->
+  <!-- <joint name="camera_color_optical_frame_joint" type="fixed"> -->
+  <!--   <parent link= "ur3_wrist_3_link" /> -->
+  <!--   <child link = "camera_color_optical_frame" /> -->
+  <!--   <origin xyz="-0.0852237 -0.0776651 0.0608126" rpy="-0.1188682 -0.7931895 -0.0029631" /> -->
+  <!-- </joint> -->
+  <!-- Physical dimensions -->
   <joint name="camera_color_optical_frame_joint" type="fixed">
-    <parent link= "ur3_wrist_3_link" />
-    <child link = "camera_color_optical_frame" />
-    <origin xyz="-0.0852237 -0.0776651 0.0608126" rpy="-0.1188682 -0.7931895 -0.0029631" />
+    <parent link="camera_adapter_toolside" />
+    <child link ="camera_color_optical_frame" />
+    <origin xyz="0.02005 0.035 0.0" rpy="${-pi/2.0} 0.0 ${-pi/2}" />
   </joint>
   <!-- <joint name="robotiq_2f140_base_joint" type="fixed"> -->

Commit message: [refac] reorient gripper to half a turn

File: mimik_ur3_setup_description/urdf/mimik_ur3_lab3023.xacro (robot description, xacro)
@@ -146,10 +146,10 @@
     <child link = "robotiq_2f140_base_link" />
     <!-- <origin xyz="0.0 0.0 0.0" rpy="0 0 0" /> -->
-    <origin xyz="${tcp_calibration_gripper}" rpy="0 0 0" />
+    <origin xyz="${tcp_calibration_gripper}" rpy="${pi} 0 0" />
   </joint>
   <joint name="camera_adapter_robotside_joint" type="fixed">
     <parent link= "robotiq_2f140_base_link" />
     <child link = "camera_adapter_robotside" />
-    <origin xyz="0.0443 0 0.0385" rpy="0 0 0" />
+    <origin xyz="0.0443 0 -0.0385" rpy="${pi} 0 0" />
   </joint>
   <!-- Calibrated with moveit_calibration pkg -->

Commit message: Set explicitaly the tcp of the gripper
Was previously set in the robotiq 2f140 xacro file.

File: mimik_ur3_setup_description/urdf/mimik_ur3_lab3023.xacro (robot description, xacro)
@@ -172,4 +172,11 @@
   <!--   <origin xyz="${tcp_calibration_gripper}" rpy="0 0 0" /> -->
   <!-- </joint> -->
+  <!-- Tool center point origin on the fingertip end when the gripper is fully closed -->
+  <link name="robotiq_2f140_tcp" />
+  <joint name="robotiq_2f140_tcp_joint" type="fixed">
+    <origin xyz="0.24127678495 0 0" rpy="${pi} 0 0" />
+    <parent link="robotiq_2f140_base_link" />
+    <child link="robotiq_2f140_tcp" />
+  </joint>
   <link name="robotiq_2f140_tcp_cad"/>
   <joint name="robotiq_2f140_tcp_cad_joint" type="fixed">

Commit message: [refac] apply new optical frame calibration

File: mimik_ur3_setup_description/urdf/mimik_ur3_lab3023.xacro (robot description, xacro)
@@ -85,5 +85,4 @@
     <origin xyz="${0.02005/2} 0 ${-0.023/2}" rpy="0 0 0"/>
   </xacro:sensor_d415>
-  <link name="camera_color_optical_frame"/>
   <!-- 2f-140 gripper + sillicon fingertip pads -->
   <xacro:robotiq_2f_140
@@ -153,23 +152,18 @@
     <origin xyz="0.0443 0 -0.0385" rpy="${pi} 0 0" />
   </joint>
-  <!-- Calibrated with moveit_calibration pkg -->
-  <!-- Error: 0.0021 m, 0.0063 rad-->
-  <!-- <joint name="camera_color_optical_frame_joint" type="fixed"> -->
-  <!--   <parent link= "ur3_wrist_3_link" /> -->
-  <!--   <child link = "camera_color_optical_frame" /> -->
-  <!--   <origin xyz="-0.0852237 -0.0776651 0.0608126" rpy="-0.1188682 -0.7931895 -0.0029631" /> -->
-  <!-- </joint> -->
-  <!-- Physical dimensions -->
+  <!-- Calibrated with moveit_calibration pkg on 14/01/2025 (N = 5 samples)
+       Reprojection error:
+           Translation = 0.0006048 meters
+           Rotation    = 0.00143 radians
+       WARNING: in realsense launcher, set tf_publish to false or it will change this tf
+  -->
+  <link name="camera_color_optical_frame"/>
   <joint name="camera_color_optical_frame_joint" type="fixed">
-    <parent link="camera_adapter_toolside" />
-    <child link ="camera_color_optical_frame" />
-    <origin xyz="0.02005 0.035 0.0" rpy="${-pi/2.0} 0.0 ${-pi/2}" />
-  </joint>
-  <!-- <joint name="robotiq_2f140_base_joint" type="fixed"> -->
-  <!--   <parent link= "dual_gripper_coupling_toolside_left" /> -->
-  <!--   <child link = "robotiq_2f140_base_link" /> -->
-  <!--   <!-\- <origin xyz="0.0 0.0 0.0" rpy="0 0 0" /> -\-> -->
-  <!--   <origin xyz="${tcp_calibration_gripper}" rpy="0 0 0" /> -->
-  <!-- </joint> -->
+    <parent link= "ur3_wrist_3_link" />
+    <child link = "camera_color_optical_frame" />
+    <!-- The RPY given by moveit_calibration is erroneous see:
+         https://github.com/moveit/moveit_calibration/issues/132 -->
+    <origin xyz="-0.137124 -0.0522788 0.106907" rpy="0.0255219 -0.7837478 -0.0339841" />
+  </joint>
   <!-- Tool center point origin on the fingertip end when the gripper is fully closed -->
   <link name="robotiq_2f140_tcp" />

Commit message: [refac] bump precision in optical frame
We added a 20mm translation in the +Z axis to achieve better precision
in our real world setup.

File: mimik_ur3_setup_description/urdf/mimik_ur3_lab3023.xacro (robot description, xacro)
@@ -158,11 +158,19 @@
        WARNING: in realsense launcher, set tf_publish to false or it will change this tf
   -->
-  <link name="camera_color_optical_frame"/>
-  <joint name="camera_color_optical_frame_joint" type="fixed">
+  <link name="camera_color_optical_frame_pre"/>
+  <joint name="camera_color_optical_frame_pre_joint" type="fixed">
     <parent link= "ur3_wrist_3_link" />
-    <child link = "camera_color_optical_frame" />
+    <child link = "camera_color_optical_frame_pre" />
     <!-- The RPY given by moveit_calibration is erroneous see:
          https://github.com/moveit/moveit_calibration/issues/132 -->
     <origin xyz="-0.137124 -0.0522788 0.106907" rpy="0.0255219 -0.7837478 -0.0339841" />
+  </joint>
+  <link name="camera_color_optical_frame"/>
+  <joint name="camera_color_optical_frame_joint" type="fixed">
+    <parent link= "camera_color_optical_frame_pre" />
+    <child link = "camera_color_optical_frame" />
+    <!-- We add 20mm to achieve better accuracy after some test, the Charucobaord
+         board appeared elavated by ~16mm wrt. the URDF tabletop (newport_tabletop frame) -->
+    <origin xyz="0 0 0.02" rpy="0 0 0" />
   </joint>
   <!-- Tool center point origin on the fingertip end when the gripper is fully closed -->

Commit message: [refac] update calibration: pipette_tcp + camera

File: mimik_ur3_setup_description/urdf/mimik_ur3_lab3023.xacro (robot description, xacro)
@@ -77,5 +77,4 @@
     prefix="dual_gripper_coupling_"
     visual_parameters_file="$(find robotiq_description)/config/robotiq_agc_apl_159_002/visual_parameters_bbox.yaml"/>
-  <link name="pipette_tcp" />
   <!-- Mimik camera adapter attached to gripper -->
   <xacro:mimik_realsense_camera_adapter
@@ -172,5 +171,6 @@
     <!-- We add 20mm to achieve better accuracy after some test, the Charucobaord
          board appeared elavated by ~16mm wrt. the URDF tabletop (newport_tabletop frame) -->
-    <origin xyz="0 0 0.02" rpy="0 0 0" />
+    <!-- <origin xyz="0 0 0.02" rpy="0 0 0" /> -->
+    <origin xyz="0 0 0.013" rpy="0 0 0" />
   </joint>
   <!-- Tool center point origin on the fingertip end when the gripper is fully closed -->
@@ -187,20 +187,79 @@
     <origin xyz="0.24127678495 0 0" rpy="0 0 0" />
   </joint>
+  <!-- Offset mesh to match pipette_tcp link calibration -->
   <joint name="pipette_base_joint" type="fixed">
     <parent link= "dual_gripper_coupling_toolside_right" />
     <child link = "pipette_base" />
-    <origin xyz="0.0 0.0 0.0" rpy="${pi} 0.0 0.0" />
-  </joint>
-  <!-- Sanity Check -->
-  <!-- <link name="pipette_tcp_test"/> -->
-  <!-- <joint name="lol" type="fixed"> -->
-  <!--   <parent link= "ur3_tool0" /> -->
-  <!--   <child link = "pipette_tcp_test" /> -->
-  <!--   <origin xyz="0.223439 -0.00046209 0.243363" rpy="0.0 0.0 0.0" /> -->
-  <!-- </joint> -->
-  <!-- Conveniance frame -->
+    <!-- <origin xyz="0.00151316 -0.001407139 0.00353" rpy="${pi} 0.0 0.0" /> -->
+    <!-- add small offset to match real setup Z axis 1.25 mm -->
+    <origin xyz="0.00151316 -0.001407139 0.00228" rpy="${pi} 0.0 0.0" />
+  </joint>
+  <link name="pipette_tcp"/>
   <joint name="pipette_tcp_joint" type="fixed">
     <parent link= "pipette_tip" />
     <child link = "pipette_tcp" />
+    <!-- Rotate around X axis by PI
+         Change the rotation so that it matches the calibrated point
+         with a tip when adding the tip along the X axis.
+    -->
+    <origin xyz="0 0 0" rpy="-3.1415927 0.0272858 1e-7" />
+  </joint>
+  <!-- <link name="pipette_tcp_validation"/> -->
+  <!-- <joint name="pipette_tcp_validation_joint" type="fixed"> -->
+  <!--   <parent link= "pipette_tcp" /> -->
+  <!--   <child link = "pipette_tcp_validation" /> -->
+  <!--   <!-\- <origin xyz="0 0 0" rpy="${pi} 0 0" /> -\-> -->
+  <!--   <origin xyz="0.0458171 0 0" rpy="0 0 0" /> -->
+  <!-- </joint> -->
+  <!-- Calibrated with the UR3 Teach Pendant on 17/01/2025 (N = 4 samples) dowel pin located on JJ24 newport tabletop -->
+  <link name="pipette_with_tip_tcp_pre"/>
+  <joint name="pipette_with_tip_tcp_joint_pre" type="fixed">
+    <parent link= "ur3_tool0" />
+    <child link = "pipette_with_tip_tcp_pre" />
+    <!-- The rotation given by the teach pendant is wrt. the UR3 base frame
+         X = 0.26253
+         Y = -0.00353
+         Z = 0.28204
+         Axis with angle magnitude
+         RX = -1.7569
+         RY = -1.7511
+         RZ = 0.7206
+         Converted to URDF RPY:
+         R = -2.3521618
+         P = -0.0085883
+         Y = 1.5639119
+         Rotate the frame so that the +X axis points away from the pipette tip (Y=PI/2, Z=PI)
+         Currently in the newport tabletop by: -0.008388061879533032
+    -->
+    <origin xyz="0.26253 -0.00353 0.28204" rpy="1.5707963 -0.7853981 0" />
+  </joint>
+  <!-- Adjust for real world height table -->
+  <link name="pipette_with_tip_tcp"/>
+  <joint name="pipette_with_tip_tcp_joint" type="fixed">
+    <parent link= "pipette_with_tip_tcp_pre" />
+    <child link = "pipette_with_tip_tcp" />
+    <origin xyz="-0.0083 0 0" rpy="0 0 0" />
+  </joint>
+  <!-- Start from the calibrated TCP with tip and move upwards by -X units
+       Found experimentally:
+         w/  tip: -173.47mm (Base Z axis)
+         w/o tip: -219.27mm ...
+         X = 45.8mm
+         +9.2mm difference with the latest calibration in the Z axis
+         tip head
+         frame.p = KDL::Vector(0, 0, 0.0456);
+         TODO
+  -->
+  <link name="pipette_tcp_from_tool0"/>
+  <joint name="pipette_tcp_from_tool0_joint" type="fixed">
+    <parent link= "pipette_with_tip_tcp" />
+    <child link = "pipette_tcp_from_tool0" />
+    <origin xyz="-0.0458 0 0" rpy="0 0 0" />
+  </joint>
+  <!-- Conveniance frame -->
+  <link name="pipette_tcp_old"/>
+  <joint name="pipette_tcp_old_joint" type="fixed">
+    <parent link= "pipette_tip" />
+    <child link = "pipette_tcp_old" />
     <!-- Calibrated on Apr 18 2024 with Tool Point Calibration ROS package -->
     <!-- Calibration captured 4 tool poses (out of 4 requested). Computing calibration... -->
