Commit message: [refac] use ur generic name for joint/link

File: mimik_robot_setup_description/urdf/mimik_ur3_lab3023.xacro (robot description, xacro)
@@ -2,5 +2,5 @@
 <robot name="mimik_ur3_lab3023" xmlns:xacro="http://ros.org/wiki/xacro" >
   <xacro:include filename="$(find mimik_description)/urdf/newport/vh3660_48x48_macro.xacro"/>
-  <xacro:include filename="$(find mimik_description)/urdf/mimik/ur3_big_mounting_plate_macro.xacro"/>
+  <xacro:include filename="$(find mimik_description)/urdf/mimik/ur_big_mounting_plate_macro.xacro"/>
   <xacro:include filename="$(find ur_description)/urdf/inc/ur3_macro.xacro"/>
   <xacro:include filename="$(find robotiq_description)/urdf/robotiq_fts_300_cpl_062/robotiq_fts_300_cpl_062_macro.xacro"/>
@@ -59,13 +59,11 @@
   <xacro:newport_vh3660_48x48
     prefix="newport_"/>
-  <xacro:mimik_ur3_big_mounting_plate
-    prefix="ur3_mounting_plate_"/>
+  <xacro:mimik_ur_big_mounting_plate
+    prefix="ur_mounting_plate_"/>
   <!-- UR3 with S/N: 2017333047 -->
-  <xacro:ur5_robot
-    prefix="ur3_" />
-  <!-- <xacro:ur3_robot -->
-  <!--   prefix="ur3_" -->
-  <!--   kinematics_parameters_file="$(find mimik_ur_launch)/etc/ur3-2017333047-calibration.yaml" -->
-  <!--   visual_parameters_file="$(find ur_description)/config/ur3/visual_parameters_vhacd_h16.yaml"/> -->
+  <xacro:ur3_robot
+    prefix="ur_"
+    kinematics_parameters_file="$(find mimik_ur_launch)/etc/ur3-2017333047-calibration.yaml"
+    visual_parameters_file="$(find ur_description)/config/ur3/visual_parameters_vhacd_h16.yaml"/>
   <!-- FT-300 ur coupling + sensor -->
   <xacro:robotiq_fts_300_cpl_062
@@ -115,17 +113,17 @@
     <origin xyz="0 ${-(1.6342/2.0 - 0.1/2.0)} ${2.5/2.0 - 0.0254/2.0}" rpy="0.0 0.0 0.0" />
   </joint>
-  <joint name="ur3_mounting_plate_base_joint" type="fixed">
+  <joint name="ur_mounting_plate_base_joint" type="fixed">
     <parent link= "newport_tabletop" />
-    <child link = "ur3_mounting_plate_base" />
+    <child link = "ur_mounting_plate_base" />
     <!-- Newport tabletop has matrix of 1 inch hole gap-->
     <origin xyz="${0 * 0.0254} ${-1 * 0.0254}  0.0" rpy="0.0 0.0 0.0" />
   </joint>
-  <joint name="ur3_base_joint" type="fixed">
-    <parent link= "ur3_mounting_plate_robotside" />
-    <child link = "ur3_base_link" />
+  <joint name="ur_base_joint" type="fixed">
+    <parent link= "ur_mounting_plate_robotside" />
+    <child link = "ur_base_link" />
     <origin xyz="0.0 0.0 0.0" rpy="0.0 0.0 ${pi/2}" />
   </joint>
   <joint name="robotiq_fts300_coupling_joint" type="fixed">
-    <parent link= "ur3_flange" />
+    <parent link= "ur_flange" />
     <child link = "robotiq_ft300_coupling_robotside" />
     <!-- Align mounting plate to flange -->
@@ -161,5 +159,5 @@
   <link name="camera_color_optical_frame_pre"/>
   <joint name="camera_color_optical_frame_pre_joint" type="fixed">
-    <parent link= "ur3_wrist_3_link" />
+    <parent link= "ur_wrist_3_link" />
     <child link = "camera_color_optical_frame_pre" />
     <!-- The RPY given by moveit_calibration is erroneous see:
@@ -217,5 +215,5 @@
   <link name="pipette_with_tip_tcp_pre"/>
   <joint name="pipette_with_tip_tcp_joint_pre" type="fixed">
-    <parent link= "ur3_tool0" />
+    <parent link= "ur_tool0" />
     <child link = "pipette_with_tip_tcp_pre" />
     <!-- The rotation given by the teach pendant is wrt. the UR3 base frame

File: mimik_ur3_lab3023_moveit_config/config/gazebo_mimik_ur3_lab3023.urdf (robot description, URDF)
Before this commit: robot mimik_ur3_lab3023, 52 links, 51 joints
Links:
- removed link ur3_base
- removed link ur3_base_link
- removed link ur3_base_link_inertia
- removed link ur3_flange
- removed link ur3_forearm_link
- removed link ur3_mounting_plate_base
- removed link ur3_mounting_plate_robotside
- removed link ur3_shoulder_link
- removed link ur3_tool0
- removed link ur3_upper_arm_link
- removed link ur3_wrist_1_link
- removed link ur3_wrist_2_link
- removed link ur3_wrist_3_link
- added link ur_base
- added link ur_base_link
- added link ur_base_link_inertia, mass 2.0; collision mesh filename=package://ur_description/meshes/ur3/collision/vhacd_h16/bas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; visual mesh filename=package://ur_description/meshes/ur3/visual/base.dae
- added link ur_flange
- added link ur_forearm_link, mass 1.26; collision mesh filename=package://ur_description/meshes/ur3/collision/vhacd_h16/for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; visual mesh filename=package://ur_description/meshes/ur3/visual/forearm.dae
- added link ur_mounting_plate_base, mass 0.5; collision mesh filename=package://mimik_description/meshes/mimik/ur_big_mounting_pl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; visual mesh filename=package://mimik_description/meshes/mimik/ur_big_mounting_pl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
- added link ur_mounting_plate_robotside
- added link ur_shoulder_link, mass 2.0; collision mesh filename=package://ur_description/meshes/ur3/collision/vhacd_h16/sho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; visual mesh filename=package://ur_description/meshes/ur3/visual/shoulder.dae
- added link ur_tool0
- added link ur_upper_arm_link, mass 3.42; collision mesh filename=package://ur_description/meshes/ur3/collision/vhacd_h16/upp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; visual mesh filename=package://ur_description/meshes/ur3/visual/upperarm.dae
- added link ur_wrist_1_link, mass 0.8; collision mesh filename=package://ur_description/meshes/ur3/collision/vhacd_h16/wri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; visual mesh filename=package://ur_description/meshes/ur3/visual/wrist1.dae
- added link ur_wrist_2_link, mass 0.8; collision mesh filename=package://ur_description/meshes/ur3/collision/vhacd_h16/wri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; visual mesh filename=package://ur_description/meshes/ur3/visual/wrist2.dae
- added link ur_wrist_3_link, mass 0.35; collision mesh filename=package://ur_description/meshes/ur3/collision/vhacd_h16/wri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; visual mesh filename=package://ur_description/meshes/ur3/visual/wrist3.dae
Joints:
- removed joint ur3_base_joint
- removed joint ur3_base_link-base_fixed_joint
- removed joint ur3_base_link-base_link_inertia
- removed joint ur3_elbow_joint
- removed joint ur3_flange-tool0
- removed joint ur3_mounting_plate_base_joint
- removed joint ur3_mounting_plate_robotside_joint
- removed joint ur3_shoulder_lift_joint
- removed joint ur3_shoulder_pan_joint
- removed joint ur3_wrist_1_joint
- removed joint ur3_wrist_2_joint
- removed joint ur3_wrist_3-flange
- removed joint ur3_wrist_3_joint
- added joint ur_base_joint: type fixed, parent ur_mounting_plate_robotside, child ur_base_link, origin xyz=0.0 0.0 0.0 rpy=0.0 0.0 1.5707963267948966
- added joint ur_base_link-base_fixed_joint: type fixed, parent ur_base_link, child ur_base, origin xyz=0 0 0 rpy=0 0 3.141592653589793
- added joint ur_base_link-base_link_inertia: type fixed, parent ur_base_link, child ur_base_link_inertia, origin xyz=0 0 0 rpy=0 0 3.141592653589793
- added joint ur_elbow_joint: type revolute, parent ur_upper_arm_link, child ur_forearm_link, origin xyz=-0.2436265756628402 0 0 rpy=0.0002419273107811124 -2.683708139035676e-05 -6.758303563369246e-05, axis 0 0 1, limit lower=-3.141592653589793 upper=3.141592653589793 effort=28.0 velocity=3.141592653589793
- added joint ur_flange-tool0: type fixed, parent ur_flange, child ur_tool0, origin xyz=0 0 0 rpy=1.5707963267948966 0 1.5707963267948966
- added joint ur_mounting_plate_base_joint: type fixed, parent newport_tabletop, child ur_mounting_plate_base, origin xyz=0.0 -0.0254  0.0 rpy=0.0 0.0 0.0
- added joint ur_mounting_plate_robotside_joint: type fixed, parent ur_mounting_plate_base, child ur_mounting_plate_robotside, origin xyz=0 0 0.1651 rpy=0 0 0
- added joint ur_shoulder_lift_joint: type revolute, parent ur_shoulder_link, child ur_upper_arm_link, origin xyz=2.055946359576799e-05 0 0 rpy=1.570842997539163 0 -3.478643464127787e-06, axis 0 0 1, limit lower=-6.283185307179586 upper=6.283185307179586 effort=56.0 velocity=3.141592653589793
- added joint ur_shoulder_pan_joint: type revolute, parent ur_base_link_inertia, child ur_shoulder_link, origin xyz=0 0 0.1519135963461435 rpy=0 0 2.788909693341134e-05, axis 0 0 1, limit lower=-6.283185307179586 upper=6.283185307179586 effort=56.0 velocity=3.141592653589793
- added joint ur_wrist_1_joint: type revolute, parent ur_forearm_link, child ur_wrist_1_link, origin xyz=-0.213196315637268 -0.0001470307749181737 0.1122813967685411 rpy=0.00130948398496501 0.0001103072258368812 1.022363974326258e-05, axis 0 0 1, limit lower=-6.283185307179586 upper=6.283185307179586 effort=12.0 velocity=6.283185307179586
- added joint ur_wrist_2_joint: type revolute, parent ur_wrist_1_link, child ur_wrist_2_link, origin xyz=-1.932285070751691e-05 -0.08536906110903648 -4.667877137511274e-05 rpy=1.571343114660626 0 6.090906127424239e-05, axis 0 0 1, limit lower=-6.283185307179586 upper=6.283185307179586 effort=12.0 velocity=6.283185307179586
- added joint ur_wrist_3-flange: type fixed, parent ur_wrist_3_link, child ur_flange, origin xyz=0 0 0 rpy=0 -1.5707963267948966 -1.5707963267948966
- added joint ur_wrist_3_joint: type revolute, parent ur_wrist_2_link, child ur_wrist_3_link, origin xyz=1.737185017286329e-05 0.08237703035038596 -8.107821857099018e-05 rpy=1.569812093786671 3.141592653589793 3.141588684587207, axis 0 0 1, limit lower=-6.283185307179586 upper=6.283185307179586 effort=12.0 velocity=6.283185307179586
- joint camera_color_optical_frame_joint: parent ur3_wrist_3_link -> ur_wrist_3_link
- joint robotiq_fts300_coupling_joint: parent ur3_flange -> ur_flange
