Commit message: [refac] update launch files

File: mimik_robot_setup_description/urdf/mimik_ur3_lab_mobile_capture_tool.xacro (robot description, xacro)
@@ -2,5 +2,5 @@
 <robot name="mimik_ur3_station_portable" xmlns:xacro="http://ros.org/wiki/xacro" >
   <xacro:include filename="$(find mimik_description)/urdf/newport/sa2_30x30_macro.xacro"/>
-  <xacro:include filename="$(find mimik_description)/urdf/mimik/ur3_mounting_plate_macro.xacro"/>
+  <xacro:include filename="$(find mimik_description)/urdf/mimik/ur_big_mounting_plate_macro.xacro"/>
   <xacro:include filename="$(find ur_description)/urdf/inc/ur3_macro.xacro"/>
   <xacro:include filename="$(find robotiq_description)/urdf/robotiq_fts_300_cpl_062/robotiq_fts_300_cpl_062_macro.xacro"/>
@@ -50,6 +50,6 @@
   <xacro:newport_sa2_30x30
     prefix="newport_"/>
-  <xacro:mimik_ur3_mounting_plate
-    prefix="ur3_mounting_plate_"/>
+  <xacro:mimik_ur_big_mounting_plate
+    prefix="ur_mounting_plate_"/>
   <!-- UR3 with S/N: 2017333047 -->
   <xacro:ur3_robot
@@ -77,12 +77,12 @@
     <origin xyz="${-(22 * 0.0254 - 0.0254/2)} 0 ${44*0.0254/2}" rpy="0.0 0.0 0.0" />
   </joint>
-  <joint name="ur3_mounting_plate_base_joint" type="fixed">
+  <joint name="ur_mounting_plate_base_joint" type="fixed">
     <parent link= "newport_tabletop" />
-    <child link = "ur3_mounting_plate_base" />
+    <child link = "ur_mounting_plate_base" />
     <!-- Newport tabletop has matrix of 1 inch hole gap-->
     <origin xyz="${-12 * 0.0254} ${10 * 0.0254} 0.0" rpy="0.0 0.0 ${-pi/2}" />
   </joint>
   <joint name="ur3_base_joint" type="fixed">
-    <parent link= "ur3_mounting_plate_robotside" />
+    <parent link= "ur_mounting_plate_robotside" />
     <child link = "ur3_base_link" />
     <origin xyz="0.0 0.0 0.0" rpy="0.0 0.0 0.0" />

File: mimik_robot_setup_description/urdf/mimik_ur3_lab_mobile_fts_gripper.xacro (robot description, xacro)
@@ -2,5 +2,5 @@
 <robot name="mimik_ur3_station_portable" xmlns:xacro="http://ros.org/wiki/xacro" >
   <xacro:include filename="$(find mimik_description)/urdf/newport/sa2_30x30_macro.xacro"/>
-  <xacro:include filename="$(find mimik_description)/urdf/mimik/ur3_mounting_plate_macro.xacro"/>
+  <xacro:include filename="$(find mimik_description)/urdf/mimik/ur_big_mounting_plate_macro.xacro"/>
   <xacro:include filename="$(find ur_description)/urdf/inc/ur3_macro.xacro"/>
   <xacro:include filename="$(find robotiq_description)/urdf/robotiq_fts_300_cpl_062/robotiq_fts_300_cpl_062_macro.xacro"/>
@@ -50,6 +50,6 @@
   <xacro:newport_sa2_30x30
     prefix="newport_"/>
-  <xacro:mimik_ur3_mounting_plate
-    prefix="ur3_mounting_plate_"/>
+  <xacro:mimik_ur_big_mounting_plate
+    prefix="ur_mounting_plate_"/>
   <!-- UR3 with S/N: 2017333047 -->
   <xacro:ur3_robot
@@ -81,12 +81,12 @@
     <origin xyz="${-(22 * 0.0254 - 0.0254/2)} 0 ${44*0.0254/2}" rpy="0.0 0.0 0.0" />
   </joint>
-  <joint name="ur3_mounting_plate_base_joint" type="fixed">
+  <joint name="ur_mounting_plate_base_joint" type="fixed">
     <parent link= "newport_tabletop" />
-    <child link = "ur3_mounting_plate_base" />
+    <child link = "ur_mounting_plate_base" />
     <!-- Newport tabletop has matrix of 1 inch hole gap-->
     <origin xyz="${-12 * 0.0254} ${10 * 0.0254} 0.0" rpy="0.0 0.0 ${-pi/2}" />
   </joint>
   <joint name="ur3_base_joint" type="fixed">
-    <parent link= "ur3_mounting_plate_robotside" />
+    <parent link= "ur_mounting_plate_robotside" />
     <child link = "ur3_base_link" />
     <origin xyz="0.0 0.0 0.0" rpy="0.0 0.0 0.0" />
